Commit message: comments, fix
more detailed explanation added. removed unused files.

File: src/fortyfive_robot/fortyfive_robot_description/urdf/fortyfive_robot_waffle.urdf.xacro (robot description, xacro)
@@ -17,5 +17,5 @@
       <origin xyz="-0.064 0 0.0" rpy="0 0 0"/>
       <geometry>
-        <mesh filename="package://fortyfive_robot_description/meshes/bases/waffle_base.stl" scale="0.001 0.001 0.001"/>
+        <mesh filename="package://fortyfive_robot_description/meshes/bases/waffle_base_for_open_manipulator.stl" scale="0.001 0.001 0.001"/>
       </geometry>
       <material name="light_black"/>
